File: extras/runLimiter/Version 3.0/runLimiter.kicad_sch (KiCad schematic)
At the start: 15 parts, among them J1 5-20 Volts, J2 Vout, J3 Dry Contacts, K1 Relay, Q1 2N3904, Q2 2SD2023, U1 MCP1700-330, U2 ESP8266-01s

Commit message: Refactored files, replaced C1, C2 footprints
Parts:
- C1, C2: footprint Ferrite_THT:LairdTech_28C0236-0JW-10 -> Capacitor_THT:CP_Radial_Tantal_D4.5mm_P2.50mm
Changed lines of the file:
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@@
       (effects (font (size 1.27 1.27)) (justify left))
     )
-    (property "Footprint" "Ferrite_THT:LairdTech_28C0236-0JW-10" (id 2) (at 102.87 68.58 0)
+    (property "Footprint" "Capacitor_THT:CP_Radial_Tantal_D4.5mm_P2.50mm" (id 2) (at 102.87 68.58 0)
       (effects (font (size 1.27 1.27)) hide)
     )
@@
       (effects (font (size 1.27 1.27)) (justify left))
     )
-    (property "Footprint" "Ferrite_THT:LairdTech_28C0236-0JW-10" (id 2) (at 81.28 68.58 0)
+    (property "Footprint" "Capacitor_THT:CP_Radial_Tantal_D4.5mm_P2.50mm" (id 2) (at 81.28 68.58 0)
       (effects (font (size 1.27 1.27)) hide)
     )
@@
     )
     (path "/cc62787a-f6b4-406f-80c4-9748fb60a866"
-      (reference "C1") (unit 1) (value "1.0") (footprint "Ferrite_THT:LairdTech_28C0236-0JW-10")
+      (reference "C1") (unit 1) (value "1.0") (footprint "Capacitor_THT:CP_Radial_Tantal_D4.5mm_P2.50mm")
     )
     (path "/4ed0e1ae-67a2-4420-9b0a-f45e81ac87f4"
-      (reference "C2") (unit 1) (value "1.0") (footprint "Ferrite_THT:LairdTech_28C0236-0JW-10")
+      (reference "C2") (unit 1) (value "1.0") (footprint "Capacitor_THT:CP_Radial_Tantal_D4.5mm_P2.50mm")
     )
     (path "/7d0a833c-82ce-4ebd-a370-b006de4fb1f1"

Commit message: Changes to board and schematic
Parts:
- removed J3: Dry Contacts, Connector_PinHeader_2.54mm:PinHeader_1x02_P2.54mm_Vertical, symbol Connector_TH_Headers:Conn_01x02
- added D2: 1N4003, Diode_THT:D_DO-41_SOD81_P10.16mm_Horizontal, symbol Diode:1N4003
- added J3: Dry Contacts, Connector_PinHeader_2.54mm:PinHeader_1x03_P2.54mm_Vertical, symbol Connector_Generic:Conn_01x03
- U1: value MCP1700-330 -> MCP1702T-3302E/TO
Connections:
- net Control Ground: now also D2.2 (A)
- net Control Power: now also D2.1 (K)
- net at K1.1: now also J3.2 (Pin_2)
- net at K1.3: now also J3.1 (Pin_1)
- net at K1.4: now also J3.3 (Pin_3)
- no-connect marks 4 -> 3
Other:
- moved on the sheet: K1
